File: ta-comm/kicad/ta-comm.kicad_pcb (KiCad board)
At the start: 4 copper layers, 45 x 45 mm, 55 parts, among them IC1 CC1110F32RHHR, IC2 F2972NEGK, IC3 STA0693A, IC4 RFFM6404, J1 Conn_01x16, J2 Conn_01x16, J3 Conn_01x04, J4 A-1JB, J5 Conn_01x04, Y1 FOX924B-27

Commit message: Updates communication board PCB
Parts:
- moved C1 0.20 mm to (135.2, 109.8)
Routing:
- net GND: track 0.00 -> 48.8 mm, vias 74 -> 73
- net /TX1: track 0.00 -> 47.5 mm
- net /RF_BYP: track 0.00 -> 46.4 mm
- net /D0: track 0.00 -> 42.8 mm
- net /TX0: track 0.00 -> 42.2 mm
- net /VDD_FILT: track 0.00 -> 41.4 mm, vias 15 -> 14
- net /RF_EN: track 0.00 -> 40.7 mm
- net /CTS1: track 0.00 -> 40.4 mm
- net /RX0: track 0.00 -> 40.1 mm
- net /RX1: track 0.00 -> 38.9 mm
- net /CTS0: track 0.00 -> 38.8 mm
- net /RTS1: track 0.00 -> 37.6 mm
- net /RTS0: track 0.00 -> 35.9 mm
- net /TX_MODE: track 0.00 -> 34.8 mm
- net /PCLK: track 0.00 -> 32.2 mm
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- added copper zone on In2.Cu, net /VDD_FILT
- added copper zone on In1.Cu, net GND
Other:
- board text added: "3V3"
- board text added: "C1"
- board text added: "C10"
- board text added: "C11"
- board text added: "C12"
- board text added: "C13"
- board text added: "C14"
- board text added: "C15"
- board text added: "C16"
- board text added: "C17"
- board text added: "C18"
- board text added: "C19"
- board text added: "C2"
- board text added: "C20"
- board text added: "C3"
- board text added: "C4"
- board text added: "C5"
- board text added: "C6"
- board text added: "C7"
- board text added: "C8"
- board text added: "C9"
- board text added: "CTS0"
- board text added: "CTS1"
- board text added: "D0"
- board text added: "FB1"
- board text added: "GND"
- board text added: "IC1"
- board text added: "IC2"
- board text added: "IC3"
- board text added: "IC4"
- board text added: "J4"
- board text added: "L1"
- board text added: "L2"
- board text added: "LED1"
- board text added: "LED2"
- board text added: "NRST"
- board text added: "PCLK"
- board text added: "PDIO"
- board text added: "R 2"
- board text added: "R1"
- board text added: "R10"
- board text added: "R11"
- board text added: "R12"
- board text added: "R13"
- board text added: "R14"
- board text added: "R15"
- board text added: "R16"
- board text added: "R17"
- board text added: "R18"
- board text added: "R19"
- board text added: "R20"
- board text added: "R3"
- board text added: "R4"
- board text added: "R5"
- board text added: "R6"
- board text added: "R7"
- board text added: "R8"
- board text added: "R9"
- board text added: "RTS0"
- board text added: "RTS1"
- board text added: "RX0"
- board text added: "RX1"
- board text added: "TX0"
- board text added: "TX1"
- board text added: "Y1"
