File: ta-ctrl/kicad/sensors.sch (KiCad schematic (older format))
At the start: 12 parts, among them U4 LSM9DS1, U5 HT-GPS200.20

Commit message: Gerbers for control board
Parts:
- added R20, R21: DNP, ta-ctrl:R_0603_1608Metric_ctrl_cpy, symbol Device:R_US
Connections:
- net Vdd: now also R21.1
- net Vdd_GNSS: now also R20.1; no longer U5.4 (Vbackup)
- new net Vbackup: R20.2, R21.2, U5.4 (Vbackup)
Other:
- moved on the sheet: C5, R19
Changed lines of the file:
@@
 Text HLabel 3500 1450 0    50   Input ~ 0
 Vdd
-Text HLabel 7650 1850 0    50   Input ~ 0
+Text HLabel 6950 1850 0    50   Input ~ 0
 Vdd_GNSS
 Text HLabel 2550 2200 0    50   BiDi ~ 0
@@
 Wire Wire Line
 	8600 2600 8750 2600
-Wire Wire Line
-	8600 2600 8600 2800
-Wire Wire Line
-	8600 2800 8750 2800
-Connection ~ 8600 2600
 $Comp
 L power:GND #PWR017
 U 1 1 5F2C42B3
-P 8550 2950
-F 0 "#PWR017" H 8550 2700 50  0001 C CNN
-F 1 "GND" H 8555 2777 50  0000 C CNN
-F 2 "" H 8550 2950 50  0001 C CNN
-F 3 "" H 8550 2950 50  0001 C CNN
-	1    8550 2950
-	1    0    0    -1
-$EndComp
-Wire Wire Line
-	8550 2950 8550 2900
-Wire Wire Line
-	8550 2900 8750 2900
+P 8650 3000
+F 0 "#PWR017" H 8650 2750 50  0001 C CNN
+F 1 "GND" H 8655 2827 50  0000 C CNN
+F 2 "" H 8650 3000 50  0001 C CNN
+F 3 "" H 8650 3000 50  0001 C CNN
+	1    8650 3000
+	1    0    0    -1
+$EndComp
 $Comp
 L power:GND #PWR018
@@
 Wire Wire Line
 	9700 2800 10150 2800
-Text HLabel 7650 2700 0    50   Input ~ 0
+Text HLabel 6950 2700 0    50   Input ~ 0
 GNSS_nRST
 Wire Wire Line
-	7650 2700 8300 2700
+	6950 2700 7600 2700
 $Comp
 L pspice:CAP C5
 U 1 1 5F42F89E
-P 7850 2150
-F 0 "C5" H 8028 2196 50  0000 L CNN
-F 1 "2.2uF" H 8028 2105 50  0000 L CNN
-F 2 "ta-ctrl:C_0603_1608Metric_ctrl_cpy" H 7850 2150 50  0001 C CNN
-F 3 "~" H 7850 2150 50  0001 C CNN
-	1    7850 2150
-	1    0    0    -1
-$EndComp
-Wire Wire Line
-	7850 2400 7850 2450
-Wire Wire Line
-	7650 1850 7850 1850
-Wire Wire Line
-	7850 1900 7850 1850
-Connection ~ 7850 1850
-Wire Wire Line
-	7850 1850 8300 1850
+P 7150 2150
+F 0 "C5" H 7328 2196 50  0000 L CNN
+F 1 "2.2uF" H 7328 2105 50  0000 L CNN
+F 2 "ta-ctrl:C_0603_1608Metric_ctrl_cpy" H 7150 2150 50  0001 C CNN
+F 3 "~" H 7150 2150 50  0001 C CNN
+	1    7150 2150
+	1    0    0    -1
+$EndComp
+Wire Wire Line
+	7150 2400 7150 2450
+Wire Wire Line
+	6950 1850 7150 1850
+Wire Wire Line
+	7150 1900 7150 1850
+Connection ~ 7150 1850
+Wire Wire Line
+	7150 1850 7600 1850
 $Comp
 L Device:R_US R19
 U 1 1 5F444CC6
-P 8300 2150
-F 0 "R19" H 8368 2196 50  0000 L CNN
-F 1 "DNP" H 8368 2105 50  0000 L CNN
-F 2 "ta-ctrl:R_0603_1608Metric_ctrl_cpy" V 8340 2140 50  0001 C CNN
-F 3 "~" H 8300 2150 50  0001 C CNN
-	1    8300 2150
+P 7600 2150
+F 0 "R19" H 7668 2196 50  0000 L CNN
+F 1 "DNP" H 7668 2105 50  0000 L CNN
+F 2 "ta-ctrl:R_0603_1608Metric_ctrl_cpy" V 7640 2140 50  0001 C CNN
+F 3 "~" H 7600 2150 50  0001 C CNN
+	1    7600 2150
 	1    0    0    -1
 $EndComp
@@
 	8600 2500 8600 2600
 Wire Wire Line
-	8300 2000 8300 1850
-Connection ~ 8300 1850
-Wire Wire Line
-	8300 1850 8600 1850
-Wire Wire Line
-	8300 2300 8300 2700
-Connection ~ 8300 2700
-Wire Wire Line
-	8300 2700 8750 2700
+	7600 2000 7600 1850
+Connection ~ 7600 1850
+Wire Wire Line
+	7600 2300 7600 2700
+Connection ~ 7600 2700
 $Comp
 L Device:R_US R18
@@
 L power:GND #PWR016
 U 1 1 5F77F24C
-P 7850 2450
-F 0 "#PWR016" H 7850 2200 50  0001 C CNN
-F 1 "GND" H 7855 2277 50  0000 C CNN
-F 2 "" H 7850 2450 50  0001 C CNN
-F 3 "" H 7850 2450 50  0001 C CNN
-	1    7850 2450
+P 7150 2450
+F 0 "#PWR016" H 7150 2200 50  0001 C CNN
+F 1 "GND" H 7155 2277 50  0000 C CNN
+F 2 "" H 7150 2450 50  0001 C CNN
+F 3 "" H 7150 2450 50  0001 C CNN
+	1    7150 2450
 	1    0    0    -1
 $EndComp
@@
 	3600 3400 3700 3400
 Connection ~ 3700 3400
+$Comp
+L Device:R_US R20
+U 1 1 5F2BE1E4
+P 8000 2150
+F 0 "R20" H 8068 2196 50  0000 L CNN
+F 1 "DNP" H 8068 2105 50  0000 L CNN
+F 2 "ta-ctrl:R_0603_1608Metric_ctrl_cpy" V 8040 2140 50  0001 C CNN
+F 3 "~" H 8000 2150 50  0001 C CNN
+	1    8000 2150
+	1    0    0    -1
+$EndComp
+Wire Wire Line
+	8000 2800 8000 2300
+Wire Wire Line
+	8000 2000 8000 1850
+Wire Wire Line
+	7600 1850 8000 1850
+Connection ~ 8000 1850
+Wire Wire Line
+	8650 3000 8650 2900
+Wire Wire Line
+	8650 2900 8750 2900
+Wire Wire Line
+	8000 2800 8400 2800
+Wire Wire Line
+	7600 2700 8750 2700
+Wire Wire Line
+	8000 1850 8600 1850
+$Comp
+L Device:R_US R21
+U 1 1 5F2E260A
+P 8400 2150
+F 0 "R21" H 8468 2196 50  0000 L CNN
+F 1 "DNP" H 8468 2105 50  0000 L CNN
+F 2 "ta-ctrl:R_0603_1608Metric_ctrl_cpy" V 8440 2140 50  0001 C CNN
+F 3 "~" H 8400 2150 50  0001 C CNN
+	1    8400 2150
+	1    0    0    -1
+$EndComp
+Wire Wire Line
+	8400 2000 8400 1450
+Wire Wire Line
+	8400 1450 5550 1450
+Connection ~ 5550 1450
+Wire Wire Line
+	8400 2300 8400 2800
+Connection ~ 8400 2800
+Wire Wire Line
+	8400 2800 8750 2800
+Text Label 8100 2800 0    50   ~ 0
+Vbackup
 $EndSCHEMATC

Commit message: updated parts vendors and added BOM
Parts:
- C1: Manufacturer Part Number (none) -> C0603C103F3GACTU; Vendor (none) -> Digikey; Vendor Part Number (none) -> 399-8985-1-ND
- C2, C4: Manufacturer Part Number (none) -> C0603C104K8RACAUTO; Vendor (none) -> Digikey; Vendor Part Number (none) -> 399-17574-1-ND
- C3: Manufacturer Part Number (none) -> C1608X7S0J106M080AC; Vendor (none) -> Digikey; Vendor Part Number (none) -> 445-9104-1-ND
- C5: Manufacturer Part Number (none) -> C0603C225K8RACTU; Vendor (none) -> Digikey; Vendor Part Number (none) -> 399-11681-1-ND
- R15, R17: Manufacturer Part Number (none) -> CRCW060310K0FKEAHP; Vendor (none) -> Digikey; Vendor Part Number (none) -> 541-10.0KSCT-ND
- U4: Manufacturer Part Number (none) -> LSM9DS1TR; Vendor (none) -> Digikey; Vendor Part Number (none) -> 497-14946-1-ND
Changed lines of the file:
@@
 F 2 "ta-ctrl:LSM9DS1TRL" H 5200 3250 50  0001 C CNN
 F 3 "http://www.st.com/content/ccc/resource/technical/document/datasheet/1e/3f/2a/d6/25/eb/48/46/DM00103319.pdf/files/DM00103319.pdf/jcr:content/translations/en.DM00103319.pdf" H 3700 2600 50  0001 C CNN
+F 4 "LSM9DS1TR" H 3700 2500 50  0001 C CNN "Manufacturer Part Number"
+F 5 "Digikey" H 3700 2500 50  0001 C CNN "Vendor"
+F 6 "497-14946-1-ND" H 3700 2500 50  0001 C CNN "Vendor Part Number"
 	1    3700 2500
 	1    0    0    -1
@@
 F 1 "10uF" H 5178 1655 50  0000 L CNN
 F 2 "ta-ctrl:C_0603_1608Metric_ctrl_cpy" H 5000 1700 50  0001 C CNN
-F 3 "~" H 5000 1700 50  0001 C CNN
+F 3 "https://product.tdk.com/info/en/catalog/datasheets/mlcc_commercial_general_en.pdf" H 5000 1700 50  0001 C CNN
+F 4 "C1608X7S0J106M080AC" H 5000 1700 50  0001 C CNN "Manufacturer Part Number"
+F 5 "Digikey" H 5000 1700 50  0001 C CNN "Vendor"
+F 6 "445-9104-1-ND" H 5000 1700 50  0001 C CNN "Vendor Part Number"
 	1    5000 1700
 	1    0    0    -1
@@
 F 1 "100nF" H 5728 1655 50  0000 L CNN
 F 2 "ta-ctrl:C_0603_1608Metric_ctrl_cpy" H 5550 1700 50  0001 C CNN
-F 3 "~" H 5550 1700 50  0001 C CNN
+F 3 "https://content.kemet.com/datasheets/KEM_C1023_X7R_AUTO_SMD.pdf" H 5550 1700 50  0001 C CNN
+F 4 "C0603C104K8RACAUTO" H 5550 1700 50  0001 C CNN "Manufacturer Part Number"
+F 5 "Digikey" H 5550 1700 50  0001 C CNN "Vendor"
+F 6 "399-17574-1-ND" H 5550 1700 50  0001 C CNN "Vendor Part Number"
 	1    5550 1700
 	1    0    0    -1
@@
 F 1 "10nF" H 1878 3205 50  0000 L CNN
 F 2 "ta-ctrl:C_0603_1608Metric_ctrl_cpy" H 1700 3250 50  0001 C CNN
-F 3 "~" H 1700 3250 50  0001 C CNN
+F 3 "https://content.kemet.com/datasheets/KEM_C1003_C0G_SMD.pdf" H 1700 3250 50  0001 C CNN
+F 4 "C0603C103F3GACTU" H 1700 3250 50  0001 C CNN "Manufacturer Part Number"
+F 5 "Digikey" H 1700 3250 50  0001 C CNN "Vendor"
+F 6 "399-8985-1-ND" H 1700 3250 50  0001 C CNN "Vendor Part Number"
 	1    1700 3250
 	1    0    0    -1
@@
 F 1 "100nF" H 2578 3305 50  0000 L CNN
 F 2 "ta-ctrl:C_0603_1608Metric_ctrl_cpy" H 2400 3350 50  0001 C CNN
-F 3 "~" H 2400 3350 50  0001 C CNN
+F 3 "https://content.kemet.com/datasheets/KEM_C1023_X7R_AUTO_SMD.pdf" H 2400 3350 50  0001 C CNN
+F 4 "C0603C104K8RACAUTO" H 2400 3350 50  0001 C CNN "Manufacturer Part Number"
+F 5 "Digikey" H 2400 3350 50  0001 C CNN "Vendor"
+F 6 "399-17574-1-ND" H 2400 3350 50  0001 C CNN "Vendor Part Number"
 	1    2400 3350
 	1    0    0    -1
@@
 F 1 "10k" H 4618 1905 50  0000 L CNN
 F 2 "ta-ctrl:R_0603_1608Metric_ctrl_cpy" V 4590 1940 50  0001 C CNN
-F 3 "~" H 4550 1950 50  0001 C CNN
+F 3 "https://www.digikey.com/product-detail/en/vishay-dale/CRCW060310K0FKEAHP/541-10-0KSCT-ND/2222780" H 4550 1950 50  0001 C CNN
+F 4 "CRCW060310K0FKEAHP" H 4550 1950 50  0001 C CNN "Manufacturer Part Number"
+F 5 "Digikey" H 4550 1950 50  0001 C CNN "Vendor"
+F 6 "541-10.0KSCT-ND" H 4550 1950 50  0001 C CNN "Vendor Part Number"
 	1    4550 1950
 	1    0    0    -1
@@
 F 1 "10k" H 2168 2205 50  0000 L CNN
 F 2 "ta-ctrl:R_0603_1608Metric_ctrl_cpy" V 2140 2240 50  0001 C CNN
-F 3 "~" H 2100 2250 50  0001 C CNN
+F 3 "https://www.digikey.com/product-detail/en/vishay-dale/CRCW060310K0FKEAHP/541-10-0KSCT-ND/2222780" H 2100 2250 50  0001 C CNN
+F 4 "CRCW060310K0FKEAHP" H 2100 2250 50  0001 C CNN "Manufacturer Part Number"
+F 5 "Digikey" H 2100 2250 50  0001 C CNN "Vendor"
+F 6 "541-10.0KSCT-ND" H 2100 2250 50  0001 C CNN "Vendor Part Number"
 	1    2100 2250
 	1    0    0    -1
@@
 F 1 "2.2uF" H 7328 2105 50  0000 L CNN
 F 2 "ta-ctrl:C_0603_1608Metric_ctrl_cpy" H 7150 2150 50  0001 C CNN
-F 3 "~" H 7150 2150 50  0001 C CNN
+F 3 "https://content.kemet.com/datasheets/KEM_C1002_X7R_SMD.pdf" H 7150 2150 50  0001 C CNN
+F 4 "C0603C225K8RACTU" H 7150 2150 50  0001 C CNN "Manufacturer Part Number"
+F 5 "Digikey" H 7150 2150 50  0001 C CNN "Vendor"
+F 6 "399-11681-1-ND" H 7150 2150 50  0001 C CNN "Vendor Part Number"
 	1    7150 2150
 	1    0    0    -1
