File: ta-base/ta-base/ta-base.kicad_pcb (KiCad board)
At the start: 2 copper layers, 64 x 58 mm, 19 parts, among them J1 PinSocket_16_base, J2 PinSocket_4_base, J3 PinSocket_5_base, J4 PinSocket_4_base, J5 PinSocket_5_base, J6 PinSocket_16_base, J7 PinSocket_5_base, J8 PinSocket_5_base, P1 Gnd_Screws, P2 Gnd_standoffs, SW1 SW_SPDT, SW2 SW_SPDT, U1 BSB008NE2LXXUMA1, U2 burn_wire

Commit message: fixed gnd bug on base plate
Connections:
- J2 pad 2: GND -> Net-(J2-Pad2)
- J2 pad 3: Net-(J2-Pad3) -> GND
- J4 pad 2: Net-(J4-Pad2) -> GND
- J4 pad 3: GND -> Net-(J4-Pad3)
